Commit message: Update cam_finger file

File: open_manipulator_pro_description/urdf/open_manipulator_pro.urdf.xacro (robot description, xacro)
@@ -238,17 +238,17 @@
       <origin xyz="0 0 0" rpy="0 0 0"/>
       <geometry>
-        <mesh filename="package://open_manipulator_pro_description/meshes/end_link.stl" scale="0.001 0.001 0.001"/>
-      </geometry>
-    </collision>
-    <visual>
-      <origin xyz="0 0 0" rpy="0 0 0"/>
-      <geometry>
-        <mesh filename="package://open_manipulator_pro_description/meshes/end_link.stl" scale="0.001 0.001 0.001"/>
-      </geometry>
-      <material name="grey"/>
-    </visual>
-    <inertial>
-      <origin xyz="0.00337 0.00000 0.00000" rpy="0 0 0"/>
-      <mass value="0.01919"/>
+        <mesh filename="package://open_manipulator_pro_description/meshes/cam_finger.stl" scale="0.001 0.001 0.001"/>
+      </geometry>
+    </collision>
+    <visual>
+      <origin xyz="0 0 0" rpy="0 0 0"/>
+      <geometry>
+        <mesh filename="package://open_manipulator_pro_description/meshes/cam_finger.stl" scale="0.001 0.001 0.001"/>
+      </geometry>
+      <material name="grey"/>
+    </visual>
+    <inertial>
+      <origin xyz="0.00000 0.00000 0.00000" rpy="0 0 0"/>
+      <mass value="0.50"/>
       <inertia ixx="1.0" ixy="0.0" ixz="0.0" iyy="1.0" iyz="0.0" izz="1.0" />
       <!--<inertia ixx="0.00000938" ixy="0.0" ixz="0.0" iyy="0.00000338" iyz="0.0" izz="0.00000635" />-->

Commit message: kinematics

File: open_manipulator_pro_description/urdf/open_manipulator_pro.urdf.xacro (robot description, xacro)
@@ -60,5 +60,5 @@
     <origin xyz="0.0 0.0 0.126" rpy="0 0 0"/>
     <axis xyz="0 0 1"/>
-    <limit velocity="6.5" effort="1000" lower="${-pi*0.5}" upper="${pi*0.5}" />
+    <limit velocity="6.5" effort="1000" lower="${-pi}" upper="${pi}" />
     <dynamics damping="0.7"/>
   </joint>

Commit message: update IK

File: open_manipulator_pro_description/urdf/open_manipulator_pro.urdf.xacro (robot description, xacro)
@@ -94,5 +94,5 @@
     <origin xyz="0.0 0.0 0.033" rpy="0 0 0"/>
     <axis xyz="0 1 0"/>
-    <limit velocity="6.5" effort="1000" lower="${-pi*0.5}" upper="${pi*0.5}" />
+    <limit velocity="6.5" effort="1000" lower="${-pi}" upper="${pi}" />
     <dynamics damping="0.7"/>
   </joint>
@@ -127,5 +127,5 @@
     <origin xyz="0.03000 0.0 0.26400" rpy="0 0 0"/>
     <axis xyz="0 1 0"/>
-    <limit velocity="6.5" effort="1000" lower="${-pi*0.5}" upper="${pi*0.5}" />
+    <limit velocity="6.5" effort="1000" lower="${-pi}" upper="${pi}" />
     <dynamics damping="0.7"/>
   </joint>
@@ -160,5 +160,5 @@
     <origin xyz="0.19500 0.0 0.03000" rpy="0 0 0"/>
     <axis xyz="1 0 0"/>
-    <limit velocity="6.5" effort="1000" lower="${-pi*0.5}" upper="${pi*0.5}" />
+    <limit velocity="6.5" effort="1000" lower="${-pi}" upper="${pi}" />
     <dynamics damping="0.7"/>
   </joint>
@@ -228,5 +228,5 @@
     <origin xyz="0.12300 0.000 0.00000" rpy="0 0 0"/>
     <axis xyz="1 0 0"/>
-    <limit velocity="6.5" effort="1000" lower="${-pi*0.5}" upper="${pi*0.5}" />
+    <limit velocity="6.5" effort="1000" lower="${-pi}" upper="${pi}" />
     <dynamics damping="0.7"/>
   </joint>
